File: hardware/schemtic_pcb/batmon.kicad_pcb (KiCad board)
At the start: 2 copper layers, 87 x 33 mm, 54 parts, among them J5 Conn_01x06, J6 Conn_01x06, J7 SW_&_LED, J8 Serial Console, J9 MCP9700, Q1 IRF3710S, Q2 2N7002, SW1 Reset, SW2 WiFi, U1 ACS712xLCTR-05B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

Commit message: Bump schematic and PCB to version 3.0
Parts:
- removed H2, H3: BAT+, MountingHole:MountingHole_3.2mm_M3_Pad
- removed H4: BAT-, MountingHole:MountingHole_3.2mm_M3_Pad
- removed JP1: SolderJumper_2_Open, Jumper:SolderJumper-2_P1.3mm_Bridged_RoundedPad1.0x1.5mm
- removed U1: ACS712xLCTR-05B, Package_SO:SOIC-8_3.9x4.9mm_P1.27mm
- added C15: 0.1uf, Capacitor_SMD:C_0603_1608Metric_Pad1.08x0.95mm_HandSolder, F.Cu at (194.0, 127.5)
- added C16: 0.1uf, Capacitor_SMD:C_0603_1608Metric_Pad1.08x0.95mm_HandSolder, F.Cu at (219.7, 104.5)
- added J1: XT60 Connector, Connector_AMASS:AMASS_XT60-F_1x02_P7.20mm_Vertical, F.Cu at (171.0, 113.1)
- added R15: 0.16R, Resistor_SMD:R_1206_3216Metric_Pad1.30x1.75mm_HandSolder, F.Cu at (180.5, 122.9)
- added R16: 0.16R, Resistor_SMD:R_1206_3216Metric_Pad1.30x1.75mm_HandSolder, F.Cu at (183.0, 122.9)
- added R17: 0.16R, Resistor_SMD:R_1206_3216Metric_Pad1.30x1.75mm_HandSolder, F.Cu at (185.5, 123.0)
- added R18: R, Resistor_SMD:R_0603_1608Metric_Pad0.98x0.95mm_HandSolder, F.Cu at (190.1, 124.5)
- added R19: 1k, Resistor_SMD:R_0603_1608Metric_Pad0.98x0.95mm_HandSolder, F.Cu at (190.1, 121.5)
- added R20: 22k, Resistor_SMD:R_0603_1608Metric_Pad0.98x0.95mm_HandSolder, F.Cu at (190.1, 127.5)
- C1: footprint Capacitor_THT:CP_Radial_D5.0mm_P2.00mm -> Capacitor_THT:CP_Radial_D10.0mm_P5.00mm
- C11: value C -> 0.1uf
- C2: value 1nf -> DNF
- C7: value 22uf -> DNF
- D1: value D_Schottky -> SS36; footprint PJA_Semiconductors:SS34_DIODE_HANDSOLDER -> Diode_SMD:D_MELF
- D4, D5: value 4V1 -> 3V9; footprint Diode_SMD:D_MELF -> Package_TO_SOT_SMD:SOT-23
- H1: value CHG- -> BAT-
- Q1: value IRF3710S -> IRF520N
- Q2: footprint Package_TO_SOT_SMD:SOT-23 -> Package_TO_SOT_SMD:TSOT-23
- R11: value 2k2 -> 1k
- R12: value 2k -> R
- R14: value 0R -> 0.16R; footprint Resistor_SMD:R_0603_1608Metric_Pad0.98x0.95mm_HandSolder -> Resistor_SMD:R_1206_3216Metric_Pad1.30x1.75mm_HandSolder
- R4: value 20k -> 22k
- U3: footprint PJA_Modules:ESP32-WROOM-32 -> RF_Module:ESP32-WROOM-32
- moved R12 20.5 mm to (196.0, 121.6), turned to 0 degrees
- moved R1 14.3 mm to (200.0, 106.5), turned to 180 degrees
- moved R14 12.4 mm to (178.0, 123.0), turned to 90 degrees
- moved U2 10.3 mm to (191.1, 103.9)
- moved C3 8.97 mm to (194.0, 129.4), turned to 180 degrees
- moved H1 8.00 mm to (169.5, 128.0)
- moved R2 7.29 mm to (196.5, 106.5)
- moved D4 6.82 mm to (221.6, 120.2)
- moved F1 6.05 mm to (171.5, 119.5), turned to 0 degrees
- moved C1 6.01 mm to (182.0, 103.1)
- moved D5 5.80 mm to (217.0, 116.4), turned to 90 degrees
- moved D1 5.15 mm to (181.0, 115.0), turned to 90 degrees
- moved C4 4.96 mm to (199.0, 113.0), turned to 180 degrees
- moved C5 4.25 mm to (186.5, 129.0), turned to 0 degrees
- moved L1 3.20 mm to (187.0, 115.0), turned to -90 degrees
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Connections:
- net /psu/BAT+ renamed /psu/CHG+
- C11 pad 1: Net-(C11-Pad1) -> BAT+SENSE
- C2 pad 1: Net-(C2-Pad1) -> AMPS_SENSE+
- C2 pad 2: GND -> Net-(C2-Pad2)
- C3 pad 1: 5V -> Net-(C2-Pad2)
- C4 pad 1: Net-(C4-Pad1) -> 5V
- D4 pad 1: Net-(C11-Pad1) -> GND
- D4 pad 2: GND -> (no net)
- D5 pad 1: TEMP1 -> GND
- D5 pad 2: GND -> (no net)
- F1 pad 1: /psu/BAT- -> /psu/CHG-
- H1 pad 1: /psu/BAT_CHARGE- -> Net-(H1-Pad1)
- J5 pad 3: AMPS_SENSE- -> BAT-SENSE
- J5 pad 4: BAT_VOLT_S -> BAT+SENSE
- J6 pad 3: AMPS_SENSE- -> BAT-SENSE
- J6 pad 4: BAT_VOLT_S -> BAT+SENSE
- L1 pad 2: Net-(C4-Pad1) -> 5V
- Q1 pad 2: Net-(Q1-Pad2) -> Net-(H1-Pad1)
- Q1 pad 3: GND -> Net-(Q1-Pad3)
- R1 pad 1: Net-(C4-Pad1) -> 5V
- R11 pad 1: Net-(C11-Pad1) -> BAT+SENSE
- R12 pad 1: BAT_VOLT_S -> Net-(C2-Pad2)
- R12 pad 2: Net-(C11-Pad1) -> BAT-SENSE
- R14 pad 1: GND -> Net-(Q1-Pad3)
- R14 pad 2: AMPS_SENSE- -> GND
- R4 pad 2: BAT_VOLT_S -> BAT+SENSE
- U5 pad 5: AMPS_SENSE- -> BAT-SENSE
- U5 pad 6: Net-(C11-Pad1) -> BAT+SENSE
Routing:
- net GND: track 256.8 -> 206.9 mm, vias 22 -> 10
- net BAT-SENSE: track 0.00 -> 43.1 mm, vias 0 -> 2
- net BAT+SENSE: track 0.00 -> 38.6 mm
- net AMPS_SENSE-: track 36.3 -> 0.00 mm, vias 1 -> 0
- net Net-(C11-Pad1): track 26.3 -> 0.00 mm, vias 2 -> 0
- net Net-(H1-Pad1): track 0.00 -> 24.4 mm
- net BAT_VOLT_S: track 24.3 -> 0.00 mm
- net Net-(C4-Pad1): track 21.2 -> 0.00 mm
- net Net-(C2-Pad2): track 0.00 -> 19.5 mm, vias 0 -> 3
- net Net-(Q1-Pad3): track 0.00 -> 15.4 mm
- net /psu/BAT_CHARGE-: track 12.9 -> 0.00 mm
- net /psu/CHG+: track 45.0 -> 35.4 mm
- net /psu/CHG-: track 0.00 -> 7.56 mm
- net 5V: track 70.0 -> 77.5 mm, vias 3 -> 2
- net /psu/BAT-: track 7.14 -> 0.00 mm
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Other:
- board text added: "CWS: Batmon V3.0"
- board text added: "Charger"
- board text added: "LED"
- board text added: "MCP9700"
- board text added: "Reset"
- board text added: "SW"
- board text added: "Serial"
- board text added: "WiFi"

Commit message: Fix unrouted R12 track that avoided DRC check
Routing:
- net Net-(C2-Pad2): track 19.5 -> 21.4 mm
Other:
- board text added: "- R12 Track missing"
- board text added: "CWS: Batmon V3.1"
- board text removed: "CWS: Batmon V3.0"
Changed lines of the file:
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@@
   )
   (paper "A4")
+  (title_block
+    (rev "3.1")
+  )
   (layers
     (0 "F.Cu" signal)
@@
     (effects (font (size 1 1) (thickness 0.15)))
   )
-  (gr_text "CWS: Batmon V3.0\n" (at 240.3 101.6) (layer "F.SilkS")
+  (gr_text "CWS: Batmon V3.1\n" (at 240.3 101.6) (layer "F.SilkS")
     (effects (font (size 1.5 1.5) (thickness 0.3)))
   )
@@
     (effects (font (size 1 1) (thickness 0.15)))
   )
+  (gr_text "- R12 Track missing" (at 173 65.1) (layer "Dwgs.User")
+    (effects (font (size 1.5 1.5) (thickness 0.3)))
+  )
   (dimension (type aligned) (layer "F.Cu")
     (pts (xy 165 132.5) (xy 206.5 132.5))
@@
   (segment (start 194.8625 129.4) (end 196.2 128.0625) (width 0.25) (layer "F.Cu") (net 51))
   (segment (start 193 122.6375) (end 193.6375 122.6375) (width 0.25) (layer "F.Cu") (net 51))
+  (segment (start 195.0875 121.6) (end 194.675 121.6) (width 0.25) (layer "F.Cu") (net 51))
+  (segment (start 194.675 121.6) (end 193.6375 122.6375) (width 0.25) (layer "F.Cu") (net 51))
   (segment (start 193 122.6375) (end 192.1375 122.6375) (width 0.25) (layer "F.Cu") (net 51))
   (segment (start 192.1375 122.6375) (end 191 121.5) (width 0.25) (layer "F.Cu") (net 51))

Commit message: - Update ADC input protextion zenners from 3V9 to 4V7 volts - Fix unrouted track - Update PCB and schemtaic to v3.1
Routing:
- net Net-(C2-Pad2): track 21.4 -> 22.0 mm
Changed lines of the file:
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@@
   (segment (start 193.6375 122.6375) (end 195 124) (width 0.25) (layer "F.Cu") (net 51))
   (segment (start 194.8625 129.4) (end 196.2 128.0625) (width 0.25) (layer "F.Cu") (net 51))
+  (segment (start 194.0375 121.6) (end 193 122.6375) (width 0.25) (layer "F.Cu") (net 51))
   (segment (start 193 122.6375) (end 193.6375 122.6375) (width 0.25) (layer "F.Cu") (net 51))
-  (segment (start 195.0875 121.6) (end 194.675 121.6) (width 0.25) (layer "F.Cu") (net 51))
-  (segment (start 194.675 121.6) (end 193.6375 122.6375) (width 0.25) (layer "F.Cu") (net 51))
+  (segment (start 195.0875 121.6) (end 194.0375 121.6) (width 0.25) (layer "F.Cu") (net 51))
   (segment (start 193 122.6375) (end 192.1375 122.6375) (width 0.25) (layer "F.Cu") (net 51))
   (segment (start 192.1375 122.6375) (end 191 121.5) (width 0.25) (layer "F.Cu") (net 51))

Commit message: - Add missing track (R12)
Other:
- board text removed: "- R12 Track missing"
Changed lines of the file:
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@@
     (effects (font (size 1 1) (thickness 0.15)))
-  )
-  (gr_text "- R12 Track missing" (at 173 65.1) (layer "Dwgs.User")
-    (effects (font (size 1.5 1.5) (thickness 0.3)))
   )
   (dimension (type aligned) (layer "F.Cu")

Commit message: Add latest schematic and PCB.
Parts:
- D4, D5: value 3V9 -> 4V7
- R12, R18: value R -> 1k
Changed lines of the file:
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@@
       (effects (font (size 1 1) (thickness 0.15)))
     )
-    (fp_text value "3V9" (at 0 2.4 180) (layer "F.Fab") hide
+    (fp_text value "4V7" (at 0 2.4 180) (layer "F.Fab") hide
       (effects (font (size 1 1) (thickness 0.15)))
     )
@@
       (effects (font (size 1 1) (thickness 0.15)))
     )
-    (fp_text value "3V9" (at 0 2.4 90) (layer "F.Fab") hide
+    (fp_text value "4V7" (at 0 2.4 90) (layer "F.Fab") hide
       (effects (font (size 1 1) (thickness 0.15)))
     )
@@
       (effects (font (size 1 1) (thickness 0.15)))
     )
-    (fp_text value "R" (at 0 1.43) (layer "F.Fab") hide
+    (fp_text value "1k" (at 0 1.43) (layer "F.Fab") hide
       (effects (font (size 1 1) (thickness 0.15)))
     )
@@
       (effects (font (size 1 1) (thickness 0.15)))
     )
-    (fp_text value "R" (at 0 1.43) (layer "F.Fab") hide
-      (effects (font (size 1 1) (thickness 0.15)))
-    )
+    (fp_text value "1k" (at 0 1.43) (layer "F.Fab") hide
+      (effects (font (size 1 1) (thickness 0.15)))
+    )
