File: hardware/schemtic_pcb/batmon.kicad_sch (KiCad schematic)
At the start: 0 parts

Commit message: Bump schematic and PCB to version 3.0
Other:
- sheet MCU ports: added BAT+SENSE, BAT-SENSE; removed AMPS_SENSE-, BAT_VOLT_S
- sheet psu ports: added BAT+SENSE, BAT-SENSE; removed AMPS_SENSE-, BAT_VOLT_S
